Commit message: added inertia to urdf

File: simple_robot_description/urdf/simple_rover.urdf (robot description, URDF)
Before this commit: robot simple_rover, 5 links, 4 joints
Links:
- link back_left_wheel: mass None -> 0.2
- link back_right_wheel: mass None -> 0.2
- link base_link: mass None -> 1.0
- link front_left_wheel: mass None -> 0.2; geometry collision cylinder length=0.04 radius=0.1; visual cylinder length=0.04 radius=0.1
- link front_right_wheel: mass None -> 0.2
